File: PCB Design/ATmega Board/PCB Design.sch (EAGLE design)
At the start: 23 parts

Commit message: worked on double sided board
Parts:
- added JP1: (no value), pinhead:PINHD-1X3
- renumbered C10 to C2, C9 to C5, R16 to R2, R17 to R1
Connections:
- net +5V: now also JP1.1
- net AREF: now also JP1.2
- net GND: now also JP1.3
Changed lines of the file:
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@@
 <parts>
 <part name="ATMEGA328P" library="Atmel_By_element14_Batch_1-00" deviceset="ATMEGA328P-PU" device=""/>
-<part name="C9" library="rcl" library_urn="urn:adsk.eagle:library:334" deviceset="C-EU" device="C0805K" value=".1uF"/>
 <part name="C3" library="rcl" library_urn="urn:adsk.eagle:library:334" deviceset="C-EU" device="C0805K" value="22pF"/>
 <part name="C4" library="rcl" library_urn="urn:adsk.eagle:library:334" deviceset="C-EU" device="C0805K" value="22pF"/>
@@
 <part name="RESET" library="switch-omron" deviceset="10-XX" device=""/>
 <part name="GND12" library="supply1" deviceset="GND" device=""/>
-<part name="R17" library="resistor" library_urn="urn:adsk.eagle:library:348" deviceset="R-EU_" device="M0805" value="10k"/>
 <part name="P+10" library="supply1" deviceset="+5V" device=""/>
 <part name="GND13" library="supply1" deviceset="GND" device=""/>
-<part name="C10" library="rcl" library_urn="urn:adsk.eagle:library:334" deviceset="C-EU" device="C0805K" value="0.33µF"/>
 <part name="P+11" library="supply1" deviceset="+5V" device=""/>
 <part name="GND14" library="supply1" deviceset="GND" device=""/>
@@
 <part name="P+14" library="supply1" deviceset="+5V" device=""/>
 <part name="GND15" library="supply1" deviceset="GND" device=""/>
-<part name="R16" library="resistor" library_urn="urn:adsk.eagle:library:348" deviceset="R-EU_" device="M0805" value="220"/>
 <part name="GND16" library="supply1" deviceset="GND" device=""/>
 <part name="R15" library="resistor" library_urn="urn:adsk.eagle:library:348" deviceset="R-EU_" device="M0805" value="220"/>
@@
 <part name="PORT_C" library="pinhead" library_urn="urn:adsk.eagle:library:325" deviceset="PINHD-1X6" device="" package3d_urn="urn:adsk.eagle:package:22472/2"/>
 <part name="JP3" library="pinhead" library_urn="urn:adsk.eagle:library:325" deviceset="PINHD-1X6" device="" package3d_urn="urn:adsk.eagle:package:22472/2"/>
+<part name="JP1" library="pinhead" library_urn="urn:adsk.eagle:library:325" deviceset="PINHD-1X3" device="" package3d_urn="urn:adsk.eagle:package:22458/2"/>
+<part name="C2" library="rcl" library_urn="urn:adsk.eagle:library:334" deviceset="C-EU" device="C0805K" value="0.33µF"/>
+<part name="R1" library="resistor" library_urn="urn:adsk.eagle:library:348" deviceset="R-EU_" device="M0805" value="10k"/>
+<part name="R2" library="resistor" library_urn="urn:adsk.eagle:library:348" deviceset="R-EU_" device="M0805" value="220"/>
+<part name="C5" library="rcl" library_urn="urn:adsk.eagle:library:334" deviceset="C-EU" device="C0805K" value=".1uF"/>
 </parts>
 <sheets>
@@
 <attribute name="VALUE" x="45.8216" y="38.8112" size="2.0828" layer="96" ratio="10" rot="SR0"/>
 </instance>
-<instance part="C9" gate="G$1" x="2.54" y="55.88"/>
 <instance part="C3" gate="G$1" x="17.78" y="10.16" smashed="yes" rot="R180">
 <attribute name="NAME" x="16.256" y="9.779" size="1.778" layer="95" rot="R180"/>
@@
 <instance part="RESET" gate="1" x="55.88" y="101.6" rot="R270"/>
 <instance part="GND12" gate="1" x="63.5" y="96.52"/>
-<instance part="R17" gate="G$1" x="55.88" y="114.3"/>
 <instance part="P+10" gate="1" x="40.64" y="114.3" smashed="yes" rot="R90">
 <attribute name="VALUE" x="45.72" y="116.84" size="1.778" layer="96" rot="R180"/>
 </instance>
 <instance part="GND13" gate="1" x="10.16" y="88.9"/>
-<instance part="C10" gate="G$1" x="7.62" y="76.2"/>
 <instance part="P+11" gate="1" x="20.32" y="96.52" smashed="yes" rot="R270">
 <attribute name="VALUE" x="15.24" y="93.98" size="1.778" layer="96"/>
@@
 <instance part="PORT_C" gate="A" x="132.08" y="45.72"/>
 <instance part="JP3" gate="A" x="132.08" y="22.86"/>
+<instance part="JP1" gate="A" x="132.08" y="5.08"/>
+<instance part="C2" gate="G$1" x="7.62" y="76.2"/>
+<instance part="R1" gate="G$1" x="55.88" y="114.3"/>
+<instance part="C5" gate="G$1" x="2.54" y="55.88"/>
 </instances>
 <busses>
@@
 </segment>
 <segment>
-<pinref part="C9" gate="G$1" pin="1"/>
 <pinref part="P+8" gate="1" pin="+5V"/>
 <wire x1="2.54" y1="58.42" x2="2.54" y2="63.5" width="0.1524" layer="91"/>
-</segment>
-<segment>
-<pinref part="R17" gate="G$1" pin="1"/>
+<pinref part="C5" gate="G$1" pin="1"/>
+</segment>
+<segment>
 <pinref part="P+10" gate="1" pin="+5V"/>
 <wire x1="43.18" y1="114.3" x2="50.8" y2="114.3" width="0.1524" layer="91"/>
+<pinref part="R1" gate="G$1" pin="1"/>
 </segment>
 <segment>
@@
 <wire x1="-12.7" y1="58.42" x2="-12.7" y2="63.5" width="0.1524" layer="91"/>
 </segment>
+<segment>
+<pinref part="JP1" gate="A" pin="1"/>
+<wire x1="129.54" y1="7.62" x2="127" y2="7.62" width="0.1524" layer="91"/>
+<label x="124.46" y="7.62" size="1.27" layer="95" rot="R180" xref="yes"/>
+</segment>
 </net>
 <net name="GND" class="0">
@@
 <segment>
 <pinref part="GND8" gate="1" pin="GND"/>
-<pinref part="C9" gate="G$1" pin="2"/>
 <wire x1="2.54" y1="45.72" x2="2.54" y2="50.8" width="0.1524" layer="91"/>
+<pinref part="C5" gate="G$1" pin="2"/>
 </segment>
 <segment>
@@
 <junction x="-17.78" y="137.16"/>
 </segment>
+<segment>
+<pinref part="JP1" gate="A" pin="3"/>
+<wire x1="129.54" y1="2.54" x2="127" y2="2.54" width="0.1524" layer="91"/>
+<label x="124.46" y="2.54" size="1.27" layer="95" rot="R180" xref="yes"/>
+</segment>
 </net>
 <net name="PB6/CRYSTAL1" class="0">
@@
 </segment>
 <segment>
-<pinref part="R17" gate="G$1" pin="2"/>
 <wire x1="60.96" y1="114.3" x2="66.04" y2="114.3" width="0.1524" layer="91"/>
 <label x="66.04" y="114.3" size="1.016" layer="95" xref="yes"/>
-</segment>
-<segment>
-<pinref part="C10" gate="G$1" pin="1"/>
+<pinref part="R1" gate="G$1" pin="2"/>
+</segment>
+<segment>
 <label x="0" y="78.74" size="1.27" layer="95" rot="R180" xref="yes"/>
 <wire x1="7.62" y1="78.74" x2="2.54" y2="78.74" width="0.1524" layer="91"/>
+<pinref part="C2" gate="G$1" pin="1"/>
 </segment>
 <segment>
@@
 <label x="35.56" y="73.66" size="1.016" layer="95" rot="R180" xref="yes"/>
 </segment>
+<segment>
+<pinref part="JP1" gate="A" pin="2"/>
+<wire x1="129.54" y1="5.08" x2="127" y2="5.08" width="0.1524" layer="91"/>
+<label x="124.46" y="5.08" size="1.27" layer="95" rot="R180" xref="yes"/>
+</segment>
 </net>
 <net name="CTS" class="0">
@@
 </segment>
 <segment>
-<pinref part="C10" gate="G$1" pin="2"/>
 <wire x1="7.62" y1="71.12" x2="2.54" y2="71.12" width="0.1524" layer="91"/>
 <label x="0" y="71.12" size="1.27" layer="95" rot="R180" xref="yes"/>
+<pinref part="C2" gate="G$1" pin="2"/>
 </segment>
 </net>
@@
 <junction x="-22.86" y="144.78"/>
 <pinref part="C1" gate="G$1" pin="+"/>
-<wire x1="-12.7" y1="157.48" x2="-12.7" y2="144.78" width="0.1524" layer="91"/>
-<junction x="-12.7" y="144.78"/>
 </segment>
 </net>
@@
 </instance>
 <instance part="GND15" gate="1" x="22.86" y="73.66" rot="R270"/>
-<instance part="R16" gate="G$1" x="7.62" y="66.04"/>
 <instance part="GND16" gate="1" x="7.62" y="58.42" rot="R270"/>
 <instance part="R15" gate="G$1" x="22.86" y="25.4" rot="R90"/>
@@
 </instance>
 <instance part="LCD" gate="G$1" x="35.56" y="48.26"/>
+<instance part="R2" gate="G$1" x="7.62" y="66.04"/>
 </instances>
 <busses>
@@
 <segment>
 <pinref part="P+14" gate="1" pin="+5V"/>
-<pinref part="R16" gate="G$1" pin="1"/>
 <wire x1="-2.54" y1="66.04" x2="2.54" y2="66.04" width="0.1524" layer="91"/>
+<pinref part="R2" gate="G$1" pin="1"/>
 </segment>
 <segment>
@@
 <net name="N$7" class="0">
 <segment>
-<pinref part="R16" gate="G$1" pin="2"/>
 <wire x1="12.7" y1="66.04" x2="25.4" y2="66.04" width="0.1524" layer="91"/>
 <pinref part="LCD" gate="G$1" pin="VDD"/>
-</segment>
-</net>
+<pinref part="R2" gate="G$1" pin="2"/>
+</segment>
+</net>

Commit message: Worked on routing and silkscreen
Parts:
- added C6: .1uF, rcl:C-EUC0805K
- renumbered ASP to USB-ASP, JP3 to PORT_B
Connections:
- net AREF: now also C6.1
- net GND: now also C6.2
Changed lines of the file:
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@@
 <part name="FTDI" library="SparkFun-Connectors" deviceset="6_PIN_SERIAL_CABLE" device="PTH"/>
 <part name="7805" library="SparkFun-IC-Power" deviceset="V_REG_78XX" device="7812" value="5V"/>
-<part name="ASP" library="SparkFun-Connectors" deviceset="AVR_SPI_PROG_5X2" device="PTH2"/>
+<part name="USB-ASP" library="SparkFun-Connectors" deviceset="AVR_SPI_PROG_5X2" device="PTH2"/>
 <part name="GND24" library="supply1" deviceset="GND" device=""/>
 <part name="P+1" library="supply1" deviceset="+5V" device=""/>
@@
 <part name="PORT_D" library="pinhead" library_urn="urn:adsk.eagle:library:325" deviceset="PINHD-1X8" device="" package3d_urn="urn:adsk.eagle:package:22409/2"/>
 <part name="PORT_C" library="pinhead" library_urn="urn:adsk.eagle:library:325" deviceset="PINHD-1X6" device="" package3d_urn="urn:adsk.eagle:package:22472/2"/>
-<part name="JP3" library="pinhead" library_urn="urn:adsk.eagle:library:325" deviceset="PINHD-1X6" device="" package3d_urn="urn:adsk.eagle:package:22472/2"/>
+<part name="PORT_B" library="pinhead" library_urn="urn:adsk.eagle:library:325" deviceset="PINHD-1X6" device="" package3d_urn="urn:adsk.eagle:package:22472/2"/>
 <part name="JP1" library="pinhead" library_urn="urn:adsk.eagle:library:325" deviceset="PINHD-1X3" device="" package3d_urn="urn:adsk.eagle:package:22458/2"/>
 <part name="C2" library="rcl" library_urn="urn:adsk.eagle:library:334" deviceset="C-EU" device="C0805K" value="0.33µF"/>
@@
 <part name="R2" library="resistor" library_urn="urn:adsk.eagle:library:348" deviceset="R-EU_" device="M0805" value="220"/>
 <part name="C5" library="rcl" library_urn="urn:adsk.eagle:library:334" deviceset="C-EU" device="C0805K" value=".1uF"/>
+<part name="C6" library="rcl" library_urn="urn:adsk.eagle:library:334" deviceset="C-EU" device="C0805K" value=".1uF"/>
+<part name="GND2" library="supply1" deviceset="GND" device=""/>
 </parts>
 <sheets>
@@
 <attribute name="VALUE" x="71.12" y="146.05" size="1.778" layer="96"/>
 </instance>
-<instance part="ASP" gate="G$1" x="-40.64" y="99.06" smashed="yes">
+<instance part="USB-ASP" gate="G$1" x="-40.64" y="99.06" smashed="yes">
 <attribute name="NAME" x="-43.18" y="107.188" size="1.778" layer="95" font="vector"/>
 <attribute name="VALUE" x="-55.626" y="85.344" size="1.778" layer="96" font="vector"/>
@@
 <instance part="PORT_D" gate="A" x="132.08" y="71.12"/>
 <instance part="PORT_C" gate="A" x="132.08" y="45.72"/>
-<instance part="JP3" gate="A" x="132.08" y="22.86"/>
+<instance part="PORT_B" gate="A" x="132.08" y="22.86"/>
 <instance part="JP1" gate="A" x="132.08" y="5.08"/>
 <instance part="C2" gate="G$1" x="7.62" y="76.2"/>
 <instance part="R1" gate="G$1" x="55.88" y="114.3"/>
 <instance part="C5" gate="G$1" x="2.54" y="55.88"/>
+<instance part="C6" gate="G$1" x="104.14" y="2.54"/>
+<instance part="GND2" gate="1" x="104.14" y="-7.62"/>
 </instances>
 <busses>
@@
 </segment>
 <segment>
-<pinref part="ASP" gate="G$1" pin="VCC"/>
+<pinref part="USB-ASP" gate="G$1" pin="VCC"/>
 <pinref part="P+1" gate="1" pin="+5V"/>
 <wire x1="-30.48" y1="104.14" x2="-27.94" y2="104.14" width="0.1524" layer="91"/>
@@
 <segment>
 <pinref part="GND24" gate="1" pin="GND"/>
-<pinref part="ASP" gate="G$1" pin="GND@4"/>
+<pinref part="USB-ASP" gate="G$1" pin="GND@4"/>
 <wire x1="-27.94" y1="93.98" x2="-30.48" y2="93.98" width="0.1524" layer="91"/>
-<pinref part="ASP" gate="G$1" pin="GND@3"/>
-<pinref part="ASP" gate="G$1" pin="GND@2"/>
+<pinref part="USB-ASP" gate="G$1" pin="GND@3"/>
+<pinref part="USB-ASP" gate="G$1" pin="GND@2"/>
 <wire x1="-30.48" y1="96.52" x2="-30.48" y2="99.06" width="0.1524" layer="91"/>
-<pinref part="ASP" gate="G$1" pin="GND@1"/>
+<pinref part="USB-ASP" gate="G$1" pin="GND@1"/>
 <wire x1="-30.48" y1="99.06" x2="-30.48" y2="101.6" width="0.1524" layer="91"/>
 <junction x="-30.48" y="99.06"/>
@@
 <label x="124.46" y="2.54" size="1.27" layer="95" rot="R180" xref="yes"/>
 </segment>
+<segment>
+<pinref part="C6" gate="G$1" pin="2"/>
+<wire x1="104.14" y1="-2.54" x2="104.14" y2="-5.08" width="0.1524" layer="91"/>
+<pinref part="GND2" gate="1" pin="GND"/>
+</segment>
 </net>
 <net name="PB6/CRYSTAL1" class="0">
@@
 </segment>
 <segment>
-<pinref part="ASP" gate="G$1" pin="RESET"/>
+<pinref part="USB-ASP" gate="G$1" pin="RESET"/>
 <wire x1="-48.26" y1="99.06" x2="-50.8" y2="99.06" width="0.1524" layer="91"/>
 <label x="-50.8" y="99.06" size="1.27" layer="95" rot="R180" xref="yes"/>
+</segment>
+<segment>
+<wire x1="45.72" y1="99.06" x2="43.18" y2="99.06" width="0.1524" layer="91"/>
+</segment>
+<segment>
+<wire x1="124.46" y1="-12.7" x2="121.92" y2="-12.7" width="0.1524" layer="91"/>
+<wire x1="129.54" y1="-12.7" x2="124.46" y2="-12.7" width="0.1524" layer="91"/>
+<junction x="124.46" y="-12.7"/>
 </segment>
 </net>
@@
 </segment>
 <segment>
-<pinref part="JP3" gate="A" pin="1"/>
+<pinref part="PORT_B" gate="A" pin="1"/>
 <wire x1="129.54" y1="30.48" x2="127" y2="30.48" width="0.1524" layer="91"/>
 <label x="124.46" y="30.48" size="1.016" layer="95" rot="R180" xref="yes"/>
@@
 </segment>
 <segment>
-<pinref part="JP3" gate="A" pin="2"/>
+<pinref part="PORT_B" gate="A" pin="2"/>
 <wire x1="129.54" y1="27.94" x2="127" y2="27.94" width="0.1524" layer="91"/>
 <label x="124.46" y="27.94" size="1.016" layer="95" rot="R180" xref="yes"/>
@@
 </segment>
 <segment>
-<pinref part="JP3" gate="A" pin="3"/>
+<pinref part="PORT_B" gate="A" pin="3"/>
 <wire x1="129.54" y1="25.4" x2="127" y2="25.4" width="0.1524" layer="91"/>
 <label x="124.46" y="25.4" size="1.016" layer="95" rot="R180" xref="yes"/>
@@
 </segment>
 <segment>
-<pinref part="ASP" gate="G$1" pin="MOSI"/>
+<pinref part="USB-ASP" gate="G$1" pin="MOSI"/>
 <wire x1="-48.26" y1="104.14" x2="-50.8" y2="104.14" width="0.1524" layer="91"/>
 <label x="-50.8" y="104.14" size="1.27" layer="95" rot="R180" xref="yes"/>
 </segment>
 <segment>
-<pinref part="JP3" gate="A" pin="4"/>
+<pinref part="PORT_B" gate="A" pin="4"/>
 <wire x1="129.54" y1="22.86" x2="127" y2="22.86" width="0.1524" layer="91"/>
 <label x="124.46" y="22.86" size="1.016" layer="95" rot="R180" xref="yes"/>
@@
 </segment>
 <segment>
-<pinref part="ASP" gate="G$1" pin="MISO"/>
+<pinref part="USB-ASP" gate="G$1" pin="MISO"/>
 <wire x1="-48.26" y1="93.98" x2="-50.8" y2="93.98" width="0.1524" layer="91"/>
 <label x="-50.8" y="93.98" size="1.27" layer="95" rot="R180" xref="yes"/>
 </segment>
 <segment>
-<pinref part="JP3" gate="A" pin="5"/>
+<pinref part="PORT_B" gate="A" pin="5"/>
 <wire x1="129.54" y1="20.32" x2="127" y2="20.32" width="0.1524" layer="91"/>
 <label x="124.46" y="20.32" size="1.016" layer="95" rot="R180" xref="yes"/>
@@
 </segment>
 <segment>
-<pinref part="ASP" gate="G$1" pin="SCK"/>
+<pinref part="USB-ASP" gate="G$1" pin="SCK"/>
 <wire x1="-48.26" y1="96.52" x2="-50.8" y2="96.52" width="0.1524" layer="91"/>
 <label x="-50.8" y="96.52" size="1.27" layer="95" rot="R180" xref="yes"/>
 </segment>
 <segment>
-<pinref part="JP3" gate="A" pin="6"/>
+<pinref part="PORT_B" gate="A" pin="6"/>
 <wire x1="129.54" y1="17.78" x2="127" y2="17.78" width="0.1524" layer="91"/>
 <label x="124.46" y="17.78" size="1.016" layer="95" rot="R180" xref="yes"/>
@@
 <wire x1="129.54" y1="5.08" x2="127" y2="5.08" width="0.1524" layer="91"/>
 <label x="124.46" y="5.08" size="1.27" layer="95" rot="R180" xref="yes"/>
+</segment>
+<segment>
+<pinref part="C6" gate="G$1" pin="1"/>
+<wire x1="104.14" y1="5.08" x2="104.14" y2="7.62" width="0.1524" layer="91"/>
+<label x="101.6" y="7.62" size="1.778" layer="95" rot="R180" xref="yes"/>
 </segment>
 </net>
@@
 </segment>
 </net>
+<net name="N$2" class="0">
+<segment>
+<wire x1="129.54" y1="-15.24" x2="124.46" y2="-15.24" width="0.1524" layer="91"/>
+</segment>
+</net>
+<net name="N$3" class="0">
+<segment>
+<wire x1="129.54" y1="-17.78" x2="124.46" y2="-17.78" width="0.1524" layer="91"/>
+</segment>
+</net>
