File: PCB Design/ATmega Board/PCB Design.sch (EAGLE design)
At the start: 25 parts

Commit message: Before routing 3.3v reg
Parts:
- added C10, C7: 10uf, resistor:CPOL-EUE2.5-6
- added JP2: (no value), pinhead:PINHD-1X2
- added JP3: (no value), pinhead:PINHD-1X6
- added U$1: V_REG_LD1117VXXLD1117-SMD, SparkFun-IC-Power:V_REG_LD1117VXXLD1117-SMD
- renumbered C12 to C9
Connections:
- removed net PC4/A4: ATMEGA328P.PC4, PORT_C.5
- removed net PC5/A5: ATMEGA328P.PC5, PORT_C.6
- new net 3.3V: C10.+, U$1.OUT
- new net N$1: C7.+, U$1.IN
- new net PC4/A4/SDA: ATMEGA328P.PC4, JP3.6, PORT_C.5
- new net PC5/A5/SCL: ATMEGA328P.PC5, JP3.5, PORT_C.6
- net +12V: now also JP2.1
- net +5V: now also JP3.1
- net AREF: now also JP3.3
- net GND: now also JP2.2, JP3.2
- net PC6/RESET: now also JP3.4
Changed lines of the file:
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@@
 <part name="P+12" library="supply1" deviceset="+5V" device=""/>
 <part name="C13" library="rcl" library_urn="urn:adsk.eagle:library:334" deviceset="C-EU" device="C0805K" value=".1uf"/>
-<part name="C12" library="resistor" deviceset="CPOL-EU" device="E2.5-6" value="10uf"/>
+<part name="C9" library="resistor" deviceset="CPOL-EU" device="E2.5-6" value="10uf"/>
 <part name="P+13" library="supply1" deviceset="+12V" device=""/>
 <part name="P+14" library="supply1" deviceset="+5V" device=""/>
@@
 <part name="C6" library="rcl" library_urn="urn:adsk.eagle:library:334" deviceset="C-EU" device="C0805K" value=".1uF"/>
 <part name="GND2" library="supply1" deviceset="GND" device=""/>
+<part name="JP2" library="pinhead" library_urn="urn:adsk.eagle:library:325" deviceset="PINHD-1X2" device="" package3d_urn="urn:adsk.eagle:package:22435/2"/>
+<part name="JP3" library="pinhead" library_urn="urn:adsk.eagle:library:325" deviceset="PINHD-1X6" device="" package3d_urn="urn:adsk.eagle:package:22472/2"/>
+<part name="U$1" library="SparkFun-IC-Power" deviceset="V_REG_LD1117VXX" device="LD1117-SMD"/>
+<part name="GND3" library="supply1" deviceset="GND" device=""/>
+<part name="C7" library="resistor" deviceset="CPOL-EU" device="E2.5-6" value="10uf"/>
+<part name="C10" library="resistor" deviceset="CPOL-EU" device="E2.5-6" value="10uf"/>
+<part name="GND4" library="supply1" deviceset="GND" device=""/>
+<part name="GND5" library="supply1" deviceset="GND" device=""/>
 </parts>
 <sheets>
@@
 <attribute name="NAME" x="64.516" y="131.699" size="1.778" layer="95" rot="R180"/>
 </instance>
-<instance part="C12" gate="G$1" x="83.82" y="139.7" smashed="yes">
+<instance part="C9" gate="G$1" x="83.82" y="139.7" smashed="yes">
 <attribute name="NAME" x="88.4174" y="135.763" size="1.778" layer="95" rot="R90"/>
 <attribute name="VALUE" x="90.9574" y="135.763" size="1.778" layer="96" rot="R90"/>
@@
 <instance part="C6" gate="G$1" x="104.14" y="2.54"/>
 <instance part="GND2" gate="1" x="104.14" y="-7.62"/>
+<instance part="JP2" gate="G$1" x="7.62" y="139.7"/>
+<instance part="JP3" gate="A" x="132.08" y="-17.78"/>
+<instance part="U$1" gate="G$1" x="71.12" y="172.72"/>
+<instance part="GND3" gate="1" x="71.12" y="160.02"/>
+<instance part="C7" gate="G$1" x="55.88" y="170.18" smashed="yes">
+<attribute name="NAME" x="60.4774" y="166.243" size="1.778" layer="95" rot="R90"/>
+<attribute name="VALUE" x="63.0174" y="166.243" size="1.778" layer="96" rot="R90"/>
+</instance>
+<instance part="C10" gate="G$1" x="83.82" y="170.18" smashed="yes">
+<attribute name="NAME" x="88.4174" y="166.243" size="1.778" layer="95" rot="R90"/>
+<attribute name="VALUE" x="90.9574" y="166.243" size="1.778" layer="96" rot="R90"/>
+</instance>
+<instance part="GND4" gate="1" x="55.88" y="160.02"/>
+<instance part="GND5" gate="1" x="83.82" y="160.02"/>
 </instances>
 <busses>
@@
 <pinref part="P+12" gate="1" pin="+5V"/>
 <wire x1="83.82" y1="142.24" x2="99.06" y2="142.24" width="0.1524" layer="91"/>
-<pinref part="C12" gate="G$1" pin="+"/>
+<pinref part="C9" gate="G$1" pin="+"/>
 <junction x="83.82" y="142.24"/>
 <pinref part="7805" gate="G$1" pin="OUT"/>
@@
 <wire x1="129.54" y1="7.62" x2="127" y2="7.62" width="0.1524" layer="91"/>
 <label x="124.46" y="7.62" size="1.27" layer="95" rot="R180" xref="yes"/>
+</segment>
+<segment>
+<pinref part="JP3" gate="A" pin="1"/>
+<wire x1="129.54" y1="-10.16" x2="127" y2="-10.16" width="0.1524" layer="91"/>
+<label x="124.46" y="-10.16" size="1.27" layer="95" rot="R180" xref="yes"/>
 </segment>
 </net>
@@
 <wire x1="71.12" y1="132.08" x2="71.12" y2="134.62" width="0.1524" layer="91"/>
 <wire x1="71.12" y1="134.62" x2="83.82" y2="134.62" width="0.1524" layer="91"/>
-<pinref part="C12" gate="G$1" pin="-"/>
+<pinref part="C9" gate="G$1" pin="-"/>
 <wire x1="83.82" y1="134.62" x2="81.28" y2="134.62" width="0.1524" layer="91"/>
 <junction x="83.82" y="134.62"/>
@@
 <wire x1="-12.7" y1="137.16" x2="-17.78" y2="137.16" width="0.1524" layer="91"/>
 <junction x="-17.78" y="137.16"/>
+<wire x1="-12.7" y1="137.16" x2="5.08" y2="137.16" width="0.1524" layer="91"/>
+<junction x="-12.7" y="137.16"/>
+<pinref part="JP2" gate="G$1" pin="2"/>
+<wire x1="5.08" y1="137.16" x2="5.08" y2="139.7" width="0.1524" layer="91"/>
 </segment>
 <segment>
@@
 <wire x1="104.14" y1="-2.54" x2="104.14" y2="-5.08" width="0.1524" layer="91"/>
 <pinref part="GND2" gate="1" pin="GND"/>
+</segment>
+<segment>
+<pinref part="JP3" gate="A" pin="2"/>
+<wire x1="129.54" y1="-12.7" x2="127" y2="-12.7" width="0.1524" layer="91"/>
+<label x="124.46" y="-12.7" size="1.27" layer="95" rot="R180" xref="yes"/>
 </segment>
 </net>
@@
 </segment>
 </net>
-<net name="PC4/A4" class="0">
+<net name="PC4/A4/SDA" class="0">
+<segment>
+<pinref part="PORT_C" gate="A" pin="5"/>
+<wire x1="129.54" y1="43.18" x2="127" y2="43.18" width="0.1524" layer="91"/>
+<label x="124.46" y="43.18" size="1.016" layer="95" rot="R180" xref="yes"/>
+</segment>
 <segment>
 <pinref part="ATMEGA328P" gate="A" pin="PC4"/>
@@
 </segment>
 <segment>
-<pinref part="PORT_C" gate="A" pin="5"/>
-<wire x1="129.54" y1="43.18" x2="127" y2="43.18" width="0.1524" layer="91"/>
-<label x="124.46" y="43.18" size="1.016" layer="95" rot="R180" xref="yes"/>
-</segment>
-</net>
-<net name="PC5/A5" class="0">
+<pinref part="JP3" gate="A" pin="6"/>
+<wire x1="129.54" y1="-22.86" x2="127" y2="-22.86" width="0.1524" layer="91"/>
+<label x="124.46" y="-22.86" size="1.27" layer="95" rot="R180" xref="yes"/>
+</segment>
+</net>
+<net name="PC5/A5/SCL" class="0">
 <segment>
 <pinref part="ATMEGA328P" gate="A" pin="PC5"/>
@@
 <wire x1="129.54" y1="40.64" x2="127" y2="40.64" width="0.1524" layer="91"/>
 <label x="124.46" y="40.64" size="1.016" layer="95" rot="R180" xref="yes"/>
+</segment>
+<segment>
+<pinref part="JP3" gate="A" pin="5"/>
+<wire x1="129.54" y1="-20.32" x2="127" y2="-20.32" width="0.1524" layer="91"/>
+<label x="124.46" y="-20.32" size="1.27" layer="95" rot="R180" xref="yes"/>
 </segment>
 </net>
@@
 </segment>
 <segment>
-<wire x1="45.72" y1="99.06" x2="43.18" y2="99.06" width="0.1524" layer="91"/>
-</segment>
-<segment>
-<wire x1="124.46" y1="-12.7" x2="121.92" y2="-12.7" width="0.1524" layer="91"/>
-<wire x1="129.54" y1="-12.7" x2="124.46" y2="-12.7" width="0.1524" layer="91"/>
-<junction x="124.46" y="-12.7"/>
+<pinref part="JP3" gate="A" pin="4"/>
+<wire x1="129.54" y1="-17.78" x2="127" y2="-17.78" width="0.1524" layer="91"/>
+<label x="124.46" y="-17.78" size="1.27" layer="95" rot="R180" xref="yes"/>
 </segment>
 </net>
@@
 <wire x1="104.14" y1="5.08" x2="104.14" y2="7.62" width="0.1524" layer="91"/>
 <label x="101.6" y="7.62" size="1.778" layer="95" rot="R180" xref="yes"/>
+</segment>
+<segment>
+<pinref part="JP3" gate="A" pin="3"/>
+<wire x1="129.54" y1="-15.24" x2="127" y2="-15.24" width="0.1524" layer="91"/>
+<label x="124.46" y="-15.24" size="1.27" layer="95" rot="R180" xref="yes"/>
 </segment>
 </net>
@@
 <junction x="-22.86" y="144.78"/>
 <pinref part="C1" gate="G$1" pin="+"/>
+<pinref part="JP2" gate="G$1" pin="1"/>
+<wire x1="5.08" y1="142.24" x2="5.08" y2="144.78" width="0.1524" layer="91"/>
+<wire x1="5.08" y1="144.78" x2="-12.7" y2="144.78" width="0.1524" layer="91"/>
+<junction x="-12.7" y="144.78"/>
 </segment>
 </net>
@@
 </segment>
 </net>
-<net name="N$2" class="0">
-<segment>
-<wire x1="129.54" y1="-15.24" x2="124.46" y2="-15.24" width="0.1524" layer="91"/>
-</segment>
-</net>
-<net name="N$3" class="0">
-<segment>
-<wire x1="129.54" y1="-17.78" x2="124.46" y2="-17.78" width="0.1524" layer="91"/>
-</segment>
-</net>
+<net name="N$1" class="0">
+<segment>
+<pinref part="U$1" gate="G$1" pin="IN"/>
+<pinref part="C7" gate="G$1" pin="+"/>
+<wire x1="63.5" y1="172.72" x2="55.88" y2="172.72" width="0.1524" layer="91"/>
+</segment>
+</net>
+<net name="3.3V" class="0">
+<segment>
+<pinref part="U$1" gate="G$1" pin="OUT"/>
+<pinref part="C10" gate="G$1" pin="+"/>
+<wire x1="78.74" y1="172.72" x2="83.82" y2="172.72" width="0.1524" layer="91"/>
+</segment>
+</net>

Commit message: Before moving pin header
Parts:
- removed C7: 10uf, resistor:CPOL-EUE2.5-6
- JP3: device pinhead:PINHD-1X6 -> pinhead:PINHD-1X7
Connections:
- removed net N$1: C7.+, U$1.IN
- net +5V: now also U$1.IN
- net 3.3V: now also JP3.3
- net AREF: now also JP3.4; no longer JP3.3
- net GND: now also C10.-, U$1.GND
- net PC4/A4/SDA: now also JP3.7; no longer JP3.6
- net PC5/A5/SCL: now also JP3.6; no longer JP3.5
- net PC6/RESET: now also JP3.5; no longer JP3.4
