File: PCB Design/ATmega Board/PCB Design.brd (EAGLE design)
At the start: 98.3 x 89.2 mm, 22 parts

Commit message: Working on design
Parts:
- removed BACKLIGHT: (no value), pinhead:1X02
- removed X1: (no value), con-ptr500:AK500/2-H
- added JP3, PORT_C: (no value), pinhead:1X06
- added PORT_D: (no value), pinhead:1X08
- moved 7805 79.9 mm to (14.7, 39.4), flipped to the bottom, turned to 270 degrees
- moved RESET 67.4 mm to (31.0, 62.2)
- moved C13 48.1 mm to (23.3, 41.7), flipped to the bottom, turned to 180 degrees
- moved FTDI 39.6 mm to (77.0, 55.9), turned to 0 degrees
- moved CONT 25.9 mm to (14.2, 44.7)
- moved C9 22.9 mm to (56.5, 37.8), flipped to the bottom, turned to 180 degrees
- moved C10 19.6 mm to (76.2, 44.2), flipped to the bottom, turned to 180 degrees
- moved R17 15.8 mm to (76.1, 41.1), flipped to the bottom, turned to 0 degrees
- moved R16 13.3 mm to (23.2, 37.1), flipped to the bottom, turned to 180 degrees
- moved 12V_JACK 7.54 mm to (24.9, 61.5), turned to 90 degrees
- moved C12 5.14 mm to (76.5, 35.3), turned to 0 degrees
- moved R15 4.37 mm to (71.9, 49.0), flipped to the bottom
- moved ASP 4.02 mm to (15.0, 25.9)
- moved C8 2.84 mm to (50.5, 29.7), flipped to the bottom, turned to 270 degrees
- flipped C3 to the bottom
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Connections:
- net CRYSTAL1 renamed PB6/CRYSTAL1
- net CRYSTAL2 renamed PB7/CRYSTAL2
- net RESET renamed PC6/RESET
- removed net A2: ATMEGA328P.25
- removed net A3: ATMEGA328P.26
- removed net A4: ATMEGA328P.27
- removed net A5: ATMEGA328P.28
- removed net D10: ATMEGA328P.16
- removed net D8: ATMEGA328P.14
- removed net D9: ATMEGA328P.15
- removed net LCD_BAK: BACKLIGHT.2, LCD.15
- removed net LCD_D4: ATMEGA328P.11, LCD.11
- removed net LCD_D5: ATMEGA328P.6, LCD.12
- removed net LCD_D6: ATMEGA328P.5, LCD.13
- removed net LCD_D7: ATMEGA328P.4, LCD.14
- removed net LCD_E: ATMEGA328P.12, LCD.6
- removed net LCD_RS: ATMEGA328P.13, LCD.4
- removed net MISO: ASP.9, ATMEGA328P.18
- removed net MOSI: ASP.1, ATMEGA328P.17
- removed net PB5/SCK: ASP.7, ATMEGA328P.19
- removed net RX: ATMEGA328P.2, FTDI.TXO
- removed net TX: ATMEGA328P.3, FTDI.RXI
- removed net V+_DIVIDED: ATMEGA328P.24
- removed net V_ACC_RESISTOR: ATMEGA328P.23
- new net PB0/D8: ATMEGA328P.14, JP3.1
- new net PB1/D9: ATMEGA328P.15, JP3.2
- new net PB2/D10: ATMEGA328P.16, JP3.3
- new net PB3/MOSI/D11: ASP.1, ATMEGA328P.17, JP3.4
- new net PB4/MISO/D12: ASP.9, ATMEGA328P.18, JP3.5
- new net PB5/SCK/D13: ASP.7, ATMEGA328P.19, JP3.6
- new net PC0/A0: ATMEGA328P.23, PORT_C.1
- new net PC1/A1: ATMEGA328P.24, PORT_C.2
- new net PC2/A2: ATMEGA328P.25, PORT_C.3
- new net PC3/A3: ATMEGA328P.26, PORT_C.4
- new net PC4/A4: ATMEGA328P.27, PORT_C.5
- new net PC5/A5: ATMEGA328P.28, PORT_C.6
- new net PD0/RX: ATMEGA328P.2, FTDI.TXO, PORT_D.1
- new net PD1/TX: ATMEGA328P.3, FTDI.RXI, PORT_D.2
- new net PD2/LCD_D7: ATMEGA328P.4, LCD.14, PORT_D.3
- new net PD3/LCD_D6: ATMEGA328P.5, LCD.13, PORT_D.4
- new net PD4/LCD_D5: ATMEGA328P.6, LCD.12, PORT_D.5
- new net PD5/LCD_D4: ATMEGA328P.11, LCD.11, PORT_D.6
- new net PD6/LCD_E: ATMEGA328P.12, LCD.6, PORT_D.7
- new net PD7/LCD_RS: ATMEGA328P.13, LCD.4, PORT_D.8
- net +12V: no longer X1.2
- net +5V: now also LCD.15; no longer BACKLIGHT.1
- net GND: no longer X1.1
Routing:
- net +5V: track 0.00 -> 204.2 mm
- net PC6/RESET: track 0.00 -> 153.2 mm
- net PB5/SCK/D13: track 0.00 -> 66.4 mm
- net PB3/MOSI/D11: track 0.00 -> 61.7 mm
- net PB4/MISO/D12: track 0.00 -> 58.7 mm
- net PD0/RX: track 0.00 -> 42.8 mm
- net N$6: track 0.00 -> 33.3 mm
- net PD1/TX: track 0.00 -> 31.2 mm
- net PB0/D8: track 0.00 -> 30.1 mm
- net +12V: track 0.00 -> 26.6 mm
- net N$14: track 0.00 -> 25.3 mm
- net PD7/LCD_RS: track 0.00 -> 25.3 mm
- net PB2/D10: track 0.00 -> 24.2 mm
- net PD6/LCD_E: track 0.00 -> 23.8 mm
- net PD5/LCD_D4: track 0.00 -> 23.1 mm
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- removed copper zone on layer 1, net GND
Other:
- board size 98.3 x 89.2 mm -> 98.3 x 66.3 mm

Commit message: testing new branch
Routing:
- net PB3/MOSI/D11: track 61.7 -> 66.3 mm
- net PB2/D10: track 24.2 -> 20.8 mm
- net PC1/A1: track 22.5 -> 20.8 mm
- net PC0/A0: track 21.9 -> 20.8 mm
Changed lines of the file:
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@@
 <contactref element="ATMEGA328P" pad="23"/>
 <contactref element="PORT_C" pad="1"/>
-<wire x1="58.166" y1="33.528" x2="58.166" y2="25.334009375" width="0.254" layer="16"/>
-<wire x1="58.166" y1="12.7" x2="58.166" y2="22.829475" width="0.254" layer="16"/>
-<wire x1="59.394271875" y1="23.455365625" x2="58.166" y2="22.829475" width="0.254" layer="16"/>
-<wire x1="59.394271875" y1="23.455365625" x2="58.166" y2="25.334009375" width="0.254" layer="16"/>
+<wire x1="58.166" y1="33.528" x2="58.166" y2="12.7" width="0.254" layer="16"/>
 </signal>
 <signal name="+12V">
@@
 <contactref element="ATMEGA328P" pad="16"/>
 <contactref element="JP3" pad="3"/>
-<wire x1="40.386" y1="18.288" x2="40.386" y2="12.7" width="0.254" layer="16"/>
-<wire x1="44.45" y1="22.352" x2="40.386" y2="18.288" width="0.254" layer="16"/>
-<wire x1="44.45" y1="24.13" x2="44.45" y2="22.352" width="0.254" layer="16"/>
-<wire x1="42.418" y1="26.162" x2="44.45" y2="24.13" width="0.254" layer="16"/>
-<wire x1="42.418" y1="31.496" x2="42.418" y2="26.162" width="0.254" layer="16"/>
-<wire x1="40.386" y1="33.528" x2="42.418" y2="31.496" width="0.254" layer="16"/>
+<wire x1="40.386" y1="33.528" x2="40.386" y2="12.7" width="0.254" layer="16"/>
 </signal>
 <signal name="PB3/MOSI/D11">
@@
 <wire x1="15.494" y1="29.718" x2="14.224" y2="30.988" width="0.254" layer="16"/>
 <wire x1="17.272" y1="29.718" x2="15.494" y2="29.718" width="0.254" layer="16"/>
-<wire x1="36.322" y1="10.668" x2="17.272" y2="29.718" width="0.254" layer="16"/>
-<wire x1="42.418" y1="10.668" x2="36.322" y2="10.668" width="0.254" layer="16"/>
-<wire x1="42.926" y1="12.7" x2="42.418" y2="10.668" width="0.254" layer="16"/>
-<wire x1="42.926" y1="26.416" x2="42.926" y2="33.528" width="0.254" layer="16"/>
-<wire x1="44.958" y1="24.384" x2="42.926" y2="26.416" width="0.254" layer="16"/>
-<wire x1="44.958" y1="14.732" x2="44.958" y2="24.384" width="0.254" layer="16"/>
-<wire x1="42.926" y1="12.7" x2="44.958" y2="14.732" width="0.254" layer="16"/>
+<wire x1="42.926" y1="33.528" x2="42.926" y2="12.7" width="0.254" layer="16"/>
+<wire x1="42.926" y1="12.7" x2="42.926" y2="11.43" width="0.254" layer="16"/>
+<wire x1="42.926" y1="11.43" x2="41.42260625" y2="11.43" width="0.254" layer="16"/>
+<wire x1="41.42260625" y1="11.43" x2="40.83840625" y2="10.8458" width="0.254" layer="16"/>
+<wire x1="40.83840625" y1="10.8458" x2="25.2222" y2="10.8458" width="0.254" layer="16"/>
+<wire x1="18.288" y1="28.702" x2="17.272" y2="29.718" width="0.254" layer="16"/>
+<wire x1="25.2222" y1="10.8458" x2="18.288" y2="17.78" width="0.254" layer="16"/>
+<wire x1="18.288" y1="17.78" x2="18.288" y2="28.702" width="0.254" layer="16"/>
 </signal>
 <signal name="PB4/MISO/D12">
@@
 <contactref element="JP3" pad="5"/>
 <wire x1="14.224" y1="20.828" x2="13.716" y2="20.828" width="0.254" layer="16"/>
-<wire x1="24.892" y1="10.16" x2="14.224" y2="20.828" width="0.254" layer="16"/>
-<wire x1="44.45" y1="10.16" x2="24.892" y2="10.16" width="0.254" layer="16"/>
-<wire x1="45.466" y1="12.7" x2="44.45" y2="10.16" width="0.254" layer="16"/>
+<wire x1="14.224" y1="20.828" x2="24.892" y2="10.16" width="0.254" layer="16"/>
 <wire x1="45.466" y1="12.7" x2="45.466" y2="33.528" width="0.254" layer="16"/>
+<wire x1="24.892" y1="10.16" x2="44.196" y2="10.16" width="0.254" layer="16"/>
+<wire x1="44.196" y1="10.16" x2="45.466" y2="11.43" width="0.254" layer="16"/>
+<wire x1="45.466" y1="11.43" x2="45.466" y2="12.7" width="0.254" layer="16"/>
 </signal>
 <signal name="PB5/SCK/D13">
@@
 <wire x1="12.446" y1="20.066" x2="12.446" y2="21.59" width="0.254" layer="16"/>
 <wire x1="22.86" y1="9.652" x2="12.446" y2="20.066" width="0.254" layer="16"/>
-<wire x1="46.482" y1="9.652" x2="22.86" y2="9.652" width="0.254" layer="16"/>
-<wire x1="48.006" y1="12.7" x2="46.482" y2="9.652" width="0.254" layer="16"/>
 <wire x1="48.006" y1="12.7" x2="48.006" y2="33.528" width="0.254" layer="16"/>
+<wire x1="48.006" y1="12.7" x2="48.006" y2="10.922" width="0.254" layer="16"/>
+<wire x1="48.006" y1="10.922" x2="46.736" y2="9.652" width="0.254" layer="16"/>
+<wire x1="46.736" y1="9.652" x2="22.86" y2="9.652" width="0.254" layer="16"/>
 </signal>
 <signal name="AREF">
@@
 <contactref element="ATMEGA328P" pad="24"/>
 <contactref element="PORT_C" pad="2"/>
-<wire x1="60.706" y1="21.082" x2="60.706" y2="12.7" width="0.254" layer="16"/>
-<wire x1="62.738" y1="23.114" x2="60.706" y2="21.082" width="0.254" layer="16"/>
-<wire x1="62.738" y1="31.496" x2="62.738" y2="23.114" width="0.254" layer="16"/>
-<wire x1="60.706" y1="33.528" x2="62.738" y2="31.496" width="0.254" layer="16"/>
+<wire x1="60.706" y1="33.528" x2="60.706" y2="12.7" width="0.254" layer="16"/>
 </signal>
 <signal name="CTS">

Commit message: worked on double sided board
Parts:
- removed C10: 0.33µF, rcl:C0805K
- removed C9: .1uF, rcl:C0805K
- removed R16: 220, resistor:M0805
- removed R17: 10k, resistor:M0805
- added C2: 0.33µF, rcl:C0805K
- added C5: .1uF, rcl:C0805K
- added JP1: (no value), pinhead:1X03
- added R1: 10k, resistor:M0805
- added R2: 220, resistor:M0805
- moved C12 15.4 mm to (82.3, 49.5)
- moved C13 12.9 mm to (20.6, 54.2), flipped to the top, turned to 270 degrees
- moved C1 0.76 mm to (13.7, 52.8), turned to 180 degrees
- moved 7805 0.51 mm to (14.7, 39.9), flipped to the top, turned to 90 degrees
- moved C8 0.25 mm to (50.5, 30.0), flipped to the top
- moved PORT_D 0.25 mm to (59.4, 55.9)
- flipped C3 to the top
- flipped C4 to the top
- flipped R15 to the top
Connections:
- net +5V: now also C5.1, JP1.1, R1.1, R2.1; no longer C9.1, R16.1, R17.1
- net AREF: now also JP1.2
- net DTR: now also C2.2; no longer C10.2
- net GND: now also C5.2, JP1.3; no longer C9.2
- net N$7: now also R2.2; no longer R16.2
- net PC6/RESET: now also C2.1, R1.2; no longer C10.1, R17.2
Routing:
- net +5V: track 204.2 -> 155.7 mm, vias 0 -> 3
- net PC6/RESET: track 153.2 -> 114.4 mm, vias 0 -> 1
- net N$14: track 25.3 -> 3.60 mm
- net AREF: track 0.00 -> 20.8 mm
- net PB4/MISO/D12: track 58.8 -> 74.3 mm
- net PB5/SCK/D13: track 66.8 -> 82.0 mm
- net +12V: track 26.6 -> 40.6 mm, vias 0 -> 1
- net PB3/MOSI/D11: track 66.3 -> 76.0 mm, vias 0 -> 1
- net DTR: track 11.8 -> 20.0 mm, vias 0 -> 1
- net PD0/RX: track 42.8 -> 35.1 mm
- net PD1/TX: track 31.2 -> 38.7 mm
- net N$6: track 33.3 -> 29.7 mm, vias 0 -> 1
- net N$7: track 16.3 -> 19.6 mm, vias 0 -> 1
- net PD7/LCD_RS: track 25.3 -> 27.6 mm
- net PD6/LCD_E: track 23.8 -> 24.9 mm
- added copper zone on layer 1, net GND
Other:
- board size 98.3 x 66.3 mm -> 98.3 x 63.8 mm

Commit message: Worked on routing and silkscreen
Parts:
- added C6: .1uF, rcl:C0805K
- moved C12 57.9 mm to (25.4, 38.6), turned to 270 degrees
- moved C5 41.6 mm to (59.7, 46.2)
- renumbered ASP to USB-ASP, JP3 to PORT_B
Connections:
- net AREF: now also C6.1
- net GND: now also C6.2
Routing:
- net AREF: track 20.8 -> 23.4 mm
- net PB3/MOSI/D11: track 76.0 -> 73.5 mm
- net +5V: track 155.7 -> 158.2 mm
- net PC6/RESET: track 114.4 -> 112.6 mm
- net N$7: track 19.6 -> 18.9 mm
Other:
- board size 98.3 x 63.8 mm -> 98.3 x 64.3 mm
- board text added: "5V"
- board text added: "AREF"
- board text added: "CTS"
- board text added: "PB0"
- board text added: "PB1"
- board text added: "PB2"
- board text added: "PB3"
- board text added: "PB4"
- board text added: "PB5"
- board text added: "PC0"
- board text added: "PC1"
- board text added: "PC2"
- board text added: "PC3"
- board text added: "PC4"
- board text added: "PC5"
- board text added: "RX"
- board text added: "TX"
- board text removed: "+"
- board text removed: "-"
- board text removed: "12/Sep/17"
- board text removed: "Chirag Shah"
- board text removed: "Constant Current Load"

Commit message: Before routing 3.3v reg
Parts:
- removed C12: 10uf, resistor:E2,5-6
- added C10, C7, C9: 10uf, resistor:E2,5-6
- added JP2: (no value), pinhead:1X02
- added JP3: (no value), pinhead:1X06
- added U$1: V_REG_LD1117VXXLD1117-SMD, SparkFun-IC-Power:SOT223
- moved C1 18.2 mm to (25.4, 38.9), turned to 90 degrees
- moved C13 17.8 mm to (21.6, 36.5)
- moved FTDI 1.52 mm to (78.5, 55.9)
- moved C2 0.76 mm to (76.2, 40.1)
Connections:
- removed net PC4/A4: ATMEGA328P.27, PORT_C.5
- removed net PC5/A5: ATMEGA328P.28, PORT_C.6
- new net 3.3V: C10.+, U$1.2
- new net N$1: C7.+, U$1.3
- new net PC4/A4/SDA: ATMEGA328P.27, JP3.6, PORT_C.5
- new net PC5/A5/SCL: ATMEGA328P.28, JP3.5, PORT_C.6
- net +12V: now also JP2.1
- net +5V: now also C9.+, JP3.1; no longer C12.+
- net AREF: now also JP3.3
- net GND: now also C9.-, JP2.2, JP3.2; no longer C12.-
- net PC6/RESET: now also JP3.4
Routing:
- net PC4/A4/SDA: track 0.00 -> 47.3 mm
- net PC5/A5/SCL: track 0.00 -> 42.3 mm
- net PC6/RESET: track 112.6 -> 149.2 mm
- net +5V: track 158.2 -> 193.8 mm, vias 3 -> 4
- net AREF: track 23.4 -> 57.1 mm
- net PC5/A5: track 20.8 -> 0.00 mm
- net PC4/A4: track 20.8 -> 0.00 mm
- net +12V: track 40.6 -> 47.2 mm, vias 1 -> 0
- net PD0/RX: track 35.5 -> 36.9 mm
- net DTR: track 20.0 -> 19.1 mm
Other:
- board text added: "RESET"
- board text added: "SCL"
- board text added: "SDA"
- board text added: "Vin"

Commit message: Before moving pin header
Parts:
- removed C7: 10uf, resistor:E2,5-6
- JP3: device pinhead:1X06 -> pinhead:1X07
- moved C10 75.6 mm to (29.7, 26.2), turned to 90 degrees
- moved U$1 47.1 mm to (13.2, 31.8), turned to 90 degrees
- moved FTDI 10.2 mm to (78.5, 66.0)
- moved PORT_D 10.2 mm to (59.4, 66.0)
- moved USB-ASP 8.57 mm to (13.2, 17.5)
- moved JP3 1.27 mm to (83.6, 12.7)
- moved C1 0.80 mm to (25.1, 38.1)
- moved 7805 0.76 mm to (14.7, 39.1)
- moved C13 0.51 mm to (21.6, 36.0)
Connections:
- removed net N$1: C7.+, U$1.3
- net +5V: now also U$1.3
- net 3.3V: now also JP3.3
- net AREF: now also JP3.4; no longer JP3.3
- net GND: now also C10.-, U$1.1
- net PC4/A4/SDA: now also JP3.7; no longer JP3.6
- net PC5/A5/SCL: now also JP3.6; no longer JP3.5
- net PC6/RESET: now also JP3.5; no longer JP3.4
Routing:
- net 3.3V: track 0.00 -> 82.7 mm, vias 0 -> 3
- net +5V: track 193.8 -> 221.7 mm, vias 4 -> 3
- net PB4/MISO/D12: track 73.9 -> 60.0 mm
- net PB5/SCK/D13: track 82.4 -> 69.4 mm
- net PD5/LCD_D4: track 22.8 -> 33.0 mm
- net PD2/LCD_D7: track 14.7 -> 24.9 mm
- net PD4/LCD_D5: track 14.7 -> 24.9 mm
- net DTR: track 19.1 -> 29.2 mm
- net PD3/LCD_D6: track 14.7 -> 24.9 mm
- net PD6/LCD_E: track 24.9 -> 35.1 mm
- net PD7/LCD_RS: track 27.6 -> 37.3 mm
- net PD1/TX: track 39.1 -> 48.6 mm
- net PB3/MOSI/D11: track 73.5 -> 66.4 mm
- net PD0/RX: track 36.9 -> 43.7 mm
- net PC6/RESET: track 149.2 -> 154.2 mm
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Other:
- board size 98.3 x 64.3 mm -> 96.3 x 64.3 mm
- board text added: "3.3V"

Commit message: Done
Parts:
- moved C9 11.7 mm to (30.0, 48.3)
- moved C1 5.06 mm to (30.0, 36.6)
- moved R15 3.87 mm to (73.4, 52.5)
- moved LCD 3.56 mm to (62.2, 37.8)
- moved JP1 2.54 mm to (53.1, 10.2)
- moved JP3 2.54 mm to (83.6, 10.2)
- moved PORT_B 2.54 mm to (41.7, 10.2)
- moved PORT_C 2.54 mm to (64.5, 10.2)
- moved C13 1.02 mm to (22.6, 36.0)
- moved C10 0.25 mm to (30.0, 26.2)
Routing:
- net +12V: track 43.2 -> 55.0 mm, vias 0 -> 1
- net +5V: track 221.7 -> 231.3 mm, vias 3 -> 4
- net N$7: track 18.9 -> 22.4 mm
- net N$6: track 29.7 -> 33.2 mm
- net 3.3V: track 82.7 -> 86.0 mm, vias 3 -> 2
- net PB0/D8: track 30.1 -> 32.6 mm
- net PC3/A3: track 20.8 -> 23.4 mm
- net PC2/A2: track 20.8 -> 23.4 mm
- net PC1/A1: track 20.8 -> 23.4 mm
- net PC0/A0: track 20.8 -> 23.4 mm
- net PB2/D10: track 20.8 -> 23.4 mm
- net PB1/D9: track 20.8 -> 23.4 mm
- net PC6/RESET: track 154.2 -> 156.5 mm
- net PC4/A4/SDA: track 49.8 -> 51.7 mm
- net N$14: track 3.60 -> 5.26 mm
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Other:
- board text added: "ATmega Board"
- board text added: "Chirag Shah 24/Feb/18"
- board text added: "PD0"
- board text added: "PD1"
- board text added: "PD2"
- board text added: "PD3"
- board text added: "PD4"
- board text added: "PD5"
- board text added: "PD6"
- board text added: "PD7"

Commit message: Corrected mistake and generated gerbers
Parts:
- moved 12V_JACK 16.8 mm to (8.38, 64.8), turned to 270 degrees
- moved RESET 2.54 mm to (31.0, 64.8)
Routing:
- net +12V: track 55.0 -> 49.2 mm
- net PC6/RESET: track 156.5 -> 159.1 mm
Changed lines of the file:
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@@
 <layer number="49" name="Reference" color="7" fill="1" visible="no" active="yes"/>
 <layer number="50" name="dxf" color="7" fill="1" visible="no" active="yes"/>
-<layer number="51" name="tDocu" color="6" fill="1" visible="no" active="yes"/>
+<layer number="51" name="tDocu" color="6" fill="1" visible="yes" active="yes"/>
 <layer number="52" name="bDocu" color="7" fill="1" visible="no" active="yes"/>
 <layer number="53" name="tGND_GNDA" color="7" fill="9" visible="no" active="no"/>
@@
 <attribute name="VALUE" x="52.07" y="47.371" size="1.27" layer="27" ratio="10" rot="R180"/>
 </element>
-<element name="RESET" library="switch-omron" package="B3F-10XX" value="" x="30.988" y="62.23" smashed="yes" rot="R270">
-<attribute name="MF" value="" x="-37.592" y="120.65" size="1.778" layer="27" rot="R270" display="off"/>
-<attribute name="MPN" value="B3F-1000" x="-37.592" y="120.65" size="1.778" layer="27" rot="R270" display="off"/>
-<attribute name="NAME" x="34.671" y="65.278" size="1.27" layer="21" ratio="10" rot="R270"/>
-<attribute name="OC_FARNELL" value="176432" x="-37.592" y="120.65" size="1.778" layer="27" rot="R270" display="off"/>
-<attribute name="OC_NEWARK" value="36M3542" x="-37.592" y="120.65" size="1.778" layer="27" rot="R270" display="off"/>
-<attribute name="VALUE" x="25.908" y="65.278" size="1.27" layer="27" ratio="10" rot="R270"/>
+<element name="RESET" library="switch-omron" package="B3F-10XX" value="" x="30.988" y="64.77" smashed="yes" rot="R270">
+<attribute name="MF" value="" x="-37.592" y="123.19" size="1.778" layer="27" rot="R270" display="off"/>
+<attribute name="MPN" value="B3F-1000" x="-37.592" y="123.19" size="1.778" layer="27" rot="R270" display="off"/>
+<attribute name="NAME" x="34.671" y="67.818" size="1.27" layer="21" ratio="10" rot="R270"/>
+<attribute name="OC_FARNELL" value="176432" x="-37.592" y="123.19" size="1.778" layer="27" rot="R270" display="off"/>
+<attribute name="OC_NEWARK" value="36M3542" x="-37.592" y="123.19" size="1.778" layer="27" rot="R270" display="off"/>
+<attribute name="VALUE" x="25.908" y="67.818" size="1.27" layer="27" ratio="10" rot="R270"/>
 </element>
 <element name="C13" library="rcl" library_urn="urn:adsk.eagle:library:334" package="C0805K" value=".1uf" x="22.606" y="35.957" smashed="yes" rot="R270">
@@
 </element>
 <element name="CONT" library="pot" library_urn="urn:adsk.eagle:library:331" package="S64W" value="50k" x="14.224" y="44.704" smashed="yes">
-<attribute name="NAME" x="8.8138" y="44.196" size="1.27" layer="21" font="vector" ratio="10" rot="R90"/>
+<attribute name="NAME" x="9.0678" y="43.688" size="1.27" layer="21" font="vector" ratio="10" rot="R90"/>
 <attribute name="VALUE" x="9.4234" y="41.783" size="1.27" layer="27" ratio="10"/>
 </element>
@@
 <attribute name="VALUE" x="48.646" y="30.972" size="1.016" layer="27" rot="R270"/>
 </element>
-<element name="12V_JACK" library="SparkFun-Connectors" package="POWER_JACK_PTH" value="POWER_JACK" x="24.892" y="61.468" smashed="yes" rot="R90">
-<attribute name="NAME" x="23.8252" y="57.8104" size="1.27" layer="21" font="vector" ratio="10" rot="R90"/>
-<attribute name="PROD_ID" value="CONN-08197" x="-9.144" y="13.462" size="1.778" layer="27" rot="R90" display="off"/>
-<attribute name="VALUE" x="24.0792" y="59.7154" size="0.6096" layer="27" font="vector" ratio="20" rot="R90"/>
+<element name="12V_JACK" library="SparkFun-Connectors" package="POWER_JACK_PTH" value="POWER_JACK" x="8.382" y="64.77" smashed="yes" rot="R270">
+<attribute name="NAME" x="24.9428" y="69.4436" size="1.27" layer="21" font="vector" ratio="10" rot="R270"/>
+<attribute name="PROD_ID" value="CONN-08197" x="42.418" y="112.776" size="1.778" layer="27" rot="R270" display="off"/>
+<attribute name="VALUE" x="9.1948" y="66.5226" size="0.6096" layer="27" font="vector" ratio="20" rot="R270"/>
 </element>
 <element name="C1" library="resistor" package="E2,5-6" value="10uf" x="29.972" y="36.576" smashed="yes" rot="R90">
@@
 <contactref element="C1" pad="+"/>
 <contactref element="JP2" pad="1"/>
-<wire x1="15.51" y1="57.15" x2="20.574" y2="57.15" width="0.8128" layer="16"/>
-<wire x1="11.192" y1="61.468" x2="15.51" y2="57.15" width="0.8128" layer="16"/>
-<wire x1="12.954" y1="54.61" x2="11.192" y2="56.372" width="0.8128" layer="16"/>
-<wire x1="11.192" y1="56.372" x2="11.192" y2="61.468" width="0.8128" layer="16"/>
-<via x="21.59" y="39.37" extent="1-16" drill="0.762"/>
-<wire x1="21.59" y1="39.37" x2="21.59" y2="56.134" width="0.8128" layer="16"/>
-<wire x1="21.59" y1="56.134" x2="20.574" y2="57.15" width="0.8128" layer="16"/>
 <wire x1="22.606" y1="36.957" x2="22.485" y2="36.836" width="0.8128" layer="1"/>
 <wire x1="22.485" y1="36.836" x2="19.532" y2="36.836" width="0.8128" layer="1"/>
-<wire x1="21.59" y1="39.37" x2="22.606" y2="38.354" width="0.8128" layer="1"/>
-<wire x1="22.606" y1="38.354" x2="22.606" y2="36.957" width="0.8128" layer="1"/>
 <wire x1="21.59" y1="36.576" x2="23.368" y2="34.798" width="0.8128" layer="16"/>
-<wire x1="21.59" y1="36.576" x2="21.59" y2="39.37" width="0.8128" layer="16"/>
 <wire x1="23.368" y1="34.798" x2="29.464" y2="34.798" width="0.8128" layer="16"/>
 <wire x1="29.464" y1="34.798" x2="29.972" y2="35.306" width="0.8128" layer="16"/>
+<wire x1="19.304" y1="54.61" x2="12.954" y2="54.61" width="0.8128" layer="16"/>
+<wire x1="22.082" y1="64.77" x2="22.082" y2="57.388" width="0.8128" layer="16"/>
+<wire x1="22.082" y1="57.388" x2="19.304" y2="54.61" width="0.8128" layer="16"/>
+<wire x1="22.485" y1="36.836" x2="22.485" y2="38.475" width="0.8128" layer="1"/>
+<wire x1="22.485" y1="38.475" x2="21.59" y2="39.37" width="0.8128" layer="1"/>
+<via x="21.59" y="39.37" extent="1-16" drill="0.8"/>
+<wire x1="21.59" y1="39.37" x2="21.59" y2="52.324" width="0.8128" layer="16"/>
+<wire x1="21.59" y1="52.324" x2="19.304" y2="54.61" width="0.8128" layer="16"/>
+<wire x1="22.485" y1="36.836" x2="21.59" y2="36.576" width="0" layer="19" extent="1-16"/>
 </signal>
 <signal name="+5V">
@@
 <wire x1="76.2" y1="41.132" x2="70.882" y2="41.132" width="0.4064" layer="1"/>
 <wire x1="70.882" y1="41.132" x2="70.866" y2="41.148" width="0.4064" layer="1"/>
-<wire x1="28.7274" y1="58.9788" x2="28.7274" y2="56.4134" width="0.4064" layer="16"/>
+<wire x1="28.7274" y1="61.5188" x2="28.7274" y2="56.4134" width="0.4064" layer="16"/>
 <wire x1="28.7274" y1="56.4134" x2="27.432" y2="55.118" width="0.4064" layer="16"/>
 <wire x1="70.866" y1="41.148" x2="70.866" y2="40.132" width="0.4064" layer="1"/>
@@
 <wire x1="26.35" y1="32.954" x2="24.892" y2="32.954" width="0.4064" layer="1"/>
 <wire x1="27.432" y1="34.036" x2="26.35" y2="32.954" width="0.4064" layer="1"/>
-<wire x1="28.7274" y1="58.9788" x2="28.7274" y2="65.4812" width="0.4064" layer="16"/>
+<wire x1="28.7274" y1="61.5188" x2="28.7274" y2="68.0212" width="0.4064" layer="16"/>
 <wire x1="11.938" y1="17.526" x2="10.16" y2="19.304" width="0.4064" layer="1"/>
 <wire x1="10.16" y1="19.304" x2="10.16" y2="23.368" width="0.4064" layer="1"/>
