File: PCB Design/ATmega Board/PCB Design.brd (EAGLE design)
At the start: 96.3 x 64.3 mm, 33 parts

Commit message: Before renumbering parts
Parts:
- removed JP3: (no value), pinhead:1X07
- removed PORT_B, PORT_C: (no value), pinhead:1X06
- removed PORT_D: (no value), pinhead:1X08
- added JP4, JP5: (no value), pinhead:2X06
- added JP6: (no value), pinhead:2X08
- added JP7: (no value), pinhead:2X03
- added R5: 330, resistor:M0805
- added RX, TX: BLUE, SparkFun-LED:LED-0603
- JP1: device pinhead:1X03 -> pinhead:2X07
- R2: value 220 -> 330
- moved R2 65.6 mm to (91.9, 53.6)
- moved JP1 30.5 mm to (83.6, 8.89)
- moved R1 2.54 mm to (27.4, 32.0)
- moved C13 1.80 mm to (24.4, 35.7)
- moved C1 0.51 mm to (30.0, 36.1)
Connections:
- new net N$3: R5.2, RX.C
- net +5V: now also JP1.2, JP7.1, JP7.2, LCD.2; no longer JP3.1, R2.1
- net 3.3V: now also JP1.5, JP1.6; no longer JP3.3
- net AREF: now also JP1.7, JP1.8, JP7.3, JP7.4; no longer JP1.2, JP3.4
- net GND: now also JP1.4, JP7.5, JP7.6, R2.1, R5.1; no longer JP3.2
- net N$7: now also TX.C; no longer LCD.2
- net PB0/D8: now also JP5.1, JP5.2; no longer PORT_B.1
- net PB1/D9: now also JP5.3, JP5.4; no longer PORT_B.2
- net PB2/D10: now also JP5.5, JP5.6; no longer PORT_B.3
- net PB3/MOSI/D11: now also JP5.7, JP5.8; no longer PORT_B.4
- net PB4/MISO/D12: now also JP5.10, JP5.9; no longer PORT_B.5
- net PB5/SCK/D13: now also JP5.11, JP5.12; no longer PORT_B.6
- net PC0/A0: now also JP4.1, JP4.2; no longer PORT_C.1
- net PC1/A1: now also JP4.3, JP4.4; no longer PORT_C.2
- net PC2/A2: now also JP4.5, JP4.6; no longer PORT_C.3
- net PC3/A3: now also JP4.7, JP4.8; no longer PORT_C.4
- net PC4/A4/SDA: now also JP1.13, JP1.14, JP4.10, JP4.9; no longer JP3.7, PORT_C.5
- net PC5/A5/SCL: now also JP1.11, JP1.12, JP4.11, JP4.12; no longer JP3.6, PORT_C.6
- net PC6/RESET: now also JP1.10, JP1.9; no longer JP3.5
- net PD0/RX: now also JP6.1, JP6.2, RX.A; no longer PORT_D.1
- net PD1/TX: now also JP6.3, JP6.4, TX.A; no longer PORT_D.2
- net PD2/LCD_D7: now also JP6.5, JP6.6; no longer PORT_D.3
- net PD3/LCD_D6: now also JP6.7, JP6.8; no longer PORT_D.4
- net PD4/LCD_D5: now also JP6.10, JP6.9; no longer PORT_D.5
- net PD5/LCD_D4: now also JP6.11, JP6.12; no longer PORT_D.6
- net PD6/LCD_E: now also JP6.13, JP6.14; no longer PORT_D.7
- net PD7/LCD_RS: now also JP6.15, JP6.16; no longer PORT_D.8
Routing:
- net PD1/TX: track 48.6 -> 72.0 mm, vias 0 -> 1
- net PD0/RX: track 43.7 -> 64.3 mm
- net +5V: track 249.6 -> 263.9 mm
- net N$3: track 0.00 -> 13.4 mm
- net N$7: track 22.4 -> 13.2 mm, vias 1 -> 0
- net PC5/A5/SCL: track 45.4 -> 50.5 mm
- net PC4/A4/SDA: track 51.7 -> 56.8 mm
- net 3.3V: track 84.7 -> 89.7 mm
- net PB5/SCK/D13: track 71.3 -> 76.2 mm
- net +12V: track 50.7 -> 55.1 mm
- net AREF: track 59.1 -> 62.6 mm
- net PB3/MOSI/D11: track 65.7 -> 68.3 mm
- net PD5/LCD_D4: track 33.0 -> 35.5 mm
- net PC3/A3: track 23.4 -> 25.9 mm
- net PC2/A2: track 23.4 -> 25.9 mm
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Other:
- board size 96.3 x 64.3 mm -> 95.8 x 64.6 mm
- board text added: "Chirag Shah 27/Feb/18"
- board text removed: "Chirag Shah 26/Feb/18"

Commit message: Final
Parts:
- removed JP7: (no value), pinhead:2X03
- added JP3: (no value), pinhead:2X06
- 1117: value (none) -> V_REG_LD1117VXXLD1117-SMD
- C10: value 10uf -> .1uF; device resistor:E2,5-6 -> rcl:C0805K
- C2: value 0.33µF -> .1uF
- C3: value 22pF -> .1uF
- C4: value 22pF -> 0.33µF
- C5, C6: value .1uF -> 22pF
- C8: value .1uF -> 10uf; device rcl:C0805K -> resistor:E2,5-6
- JP1: device pinhead:2X07 -> pinhead:1X02
- JP2: device pinhead:1X02 -> pinhead:2X08
- JP5: device pinhead:2X06 -> pinhead:2X03
- JP6: device pinhead:2X08 -> pinhead:2X07
- R1: value 10k -> 330
- R3: value 330 -> 10k
- RX, TX: value BLUE -> Yellow
- moved JP1 83.4 mm to (13.0, 53.3), turned to 270 degrees
- moved R5 81.7 mm to (22.6, 16.8), turned to 270 degrees
- moved R1 74.5 mm to (97.0, 58.7)
- moved JP6 63.2 mm to (83.6, 8.89), turned to 0 degrees
- moved JP2 48.5 mm to (59.4, 67.3), turned to 180 degrees
- moved C4 34.6 mm to (76.2, 40.1)
- moved C2 27.6 mm to (50.5, 30.0)
- moved C10 23.4 mm to (53.1, 30.0), turned to 270 degrees
- moved JP4 22.9 mm to (41.7, 8.89)
- moved C8 20.9 mm to (30.0, 26.2), turned to 90 degrees
- moved C6 19.7 mm to (42.2, 46.3)
- moved R3 15.2 mm to (27.4, 32.0), turned to 90 degrees
- moved JP5 11.4 mm to (53.1, 8.89)
- moved R2 9.58 mm to (100.1, 58.7)
- moved R4 4.32 mm to (26.9, 16.8)
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- renumbered 12V_JACK to 12V_DC, C13 to C7, CRYSTAL to Q1, LCD to LCD1, R15 to R7
Connections:
- net +12V: now also JP1.1; no longer JP2.1
- net +5V: now also C2.1, C3.1, JP5.1, JP5.2, JP6.1, JP6.2, R3.1; no longer C5.1, C8.1, JP1.1, JP1.2, JP7.1, JP7.2, R1.1
- net 3.3V: now also C8.+, JP6.5, JP6.6; no longer C10.+, JP1.5, JP1.6
- net AREF: now also C10.1, JP5.3, JP5.4, JP6.7, JP6.8; no longer C6.1, JP1.7, JP1.8, JP7.3, JP7.4
- net DTR: now also C4.2; no longer C2.2
- net GND: now also C10.2, C2.2, C3.2, C5.1, C6.1, C8.-, JP1.2, JP5.5, JP5.6, JP6.3, JP6.4, R1.1; no longer C10.-, C3.1, C4.1, C5.2, C6.2, C8.2, JP1.3, JP1.4, JP2.2, JP7.5, JP7.6, R3.1
- net N$1: now also R4.2; no longer R3.2
- net N$2: now also R5.2; no longer R4.2
- net N$3: now also R2.2; no longer R5.2
- net N$7: now also R1.2; no longer R2.2
- net PB0/D8: now also JP4.1, JP4.2; no longer JP5.1, JP5.2
- net PB1/D9: now also JP4.3, JP4.4; no longer JP5.3, JP5.4
- net PB2/D10: now also JP4.5, JP4.6; no longer JP5.5, JP5.6
- net PB3/MOSI/D11: now also JP4.7, JP4.8; no longer JP5.7, JP5.8
- net PB4/MISO/D12: now also JP4.10, JP4.9; no longer JP5.10, JP5.9
- net PB5/SCK/D13: now also JP4.11, JP4.12; no longer JP5.11, JP5.12
- net PB6/CRYSTAL1: now also C5.2; no longer C3.2
- net PB7/CRYSTAL2: now also C6.2; no longer C4.2
- net PC0/A0: now also JP3.1, JP3.2; no longer JP4.1, JP4.2
- net PC1/A1: now also JP3.3, JP3.4; no longer JP4.3, JP4.4
- net PC2/A2: now also JP3.5, JP3.6; no longer JP4.5, JP4.6
- net PC3/A3: now also JP3.7, JP3.8; no longer JP4.7, JP4.8
- net PC4/A4/SDA: now also JP3.10, JP3.9, JP6.13, JP6.14; no longer JP1.13, JP1.14, JP4.10, JP4.9
- net PC5/A5/SCL: now also JP3.11, JP3.12, JP6.11, JP6.12; no longer JP1.11, JP1.12, JP4.11, JP4.12
- net PC6/RESET: now also C4.1, JP6.10, JP6.9, R3.2; no longer C2.1, JP1.10, JP1.9, R1.2
- net PD0/RX: now also JP2.1, JP2.2; no longer JP6.1, JP6.2
- net PD1/TX: now also JP2.3, JP2.4; no longer JP6.3, JP6.4
- net PD2/LCD_D7: now also JP2.5, JP2.6; no longer JP6.5, JP6.6
- net PD3/LCD_D6: now also JP2.7, JP2.8; no longer JP6.7, JP6.8
- net PD4/LCD_D5: now also JP2.10, JP2.9; no longer JP6.10, JP6.9
- net PD5/LCD_D4: now also JP2.11, JP2.12; no longer JP6.11, JP6.12
- net PD6/LCD_E: now also JP2.13, JP2.14; no longer JP6.13, JP6.14
- net PD7/LCD_RS: now also JP2.15, JP2.16; no longer JP6.15, JP6.16
Routing:
- net N$3: track 13.4 -> 5.29 mm
- net N$7: track 13.2 -> 5.29 mm
