File: PCB Design/ATmega Board/PCB Design.brd (EAGLE design)
At the start: 95.8 x 64.6 mm, 36 parts, among them Q1 16MHz

Commit message: Corrected mistakes, V2, Final
Parts:
- moved R1 0.76 mm to (96.5, 59.4)
- moved R2 0.76 mm to (100.1, 59.4)
Connections:
- net +5V: now also RX.A, TX.A
- net GND: no longer R1.1, R2.1
- net PD0/RX: now also R2.1; no longer RX.A
- net PD1/TX: now also R1.1; no longer TX.A
Routing:
- net +5V: track 263.9 -> 279.5 mm
- net PD0/RX: track 64.3 -> 78.2 mm
- net 3.3V: track 89.7 -> 86.9 mm
- net PD1/TX: track 71.5 -> 73.1 mm
- net N$9: track 5.29 -> 4.52 mm
- net N$8: track 5.29 -> 4.52 mm
Other:
- board text added: "Chirag Shah 2/Apr/18"
- board text added: "V2"
- board text removed: "Chirag Shah 27/Feb/18"
